File: pocketchip/keys/ahole.brd (EAGLE design)
At the start: 115.6 x 77.5 mm, 0 parts

Commit message: push
Other:
- board size 115.6 x 77.5 mm -> 112.3 x 79.6 mm
Changed lines of the file:
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@@
 <layer number="27" name="tValues" color="7" fill="1" visible="yes" active="yes"/>
 <layer number="28" name="bValues" color="7" fill="1" visible="yes" active="yes"/>
-<layer number="29" name="tStop" color="7" fill="3" visible="no" active="yes"/>
+<layer number="29" name="tStop" color="7" fill="3" visible="yes" active="yes"/>
 <layer number="30" name="bStop" color="7" fill="6" visible="no" active="yes"/>
 <layer number="31" name="tCream" color="7" fill="4" visible="no" active="yes"/>
@@
 <hole x="-24.4066" y="60.48" drill="7.62"/>
 <hole x="-30.4466" y="37.7" drill="7.62"/>
-<wire x1="-58.42" y1="76.2" x2="57.15" y2="76.2" width="0.2032" layer="20"/>
-<wire x1="57.15" y1="76.2" x2="57.15" y2="-1.27" width="0.2032" layer="20"/>
-<wire x1="57.15" y1="-1.27" x2="-55.88" y2="-1.27" width="0.2032" layer="20"/>
-<wire x1="-55.88" y1="-1.27" x2="-58.42" y2="1.27" width="0.2032" layer="20"/>
-<wire x1="-58.42" y1="1.27" x2="-58.42" y2="76.2" width="0.2032" layer="20"/>
+<!-- north -->
+<wire x1="-56.134" y1="73.66" x2="56.134" y2="73.66" width="0.2032" layer="20"/>
+<!-- east -->
+<wire x1="56.134" y1="73.66" x2="56.134" y2="-5.9318" width="0.2032" layer="20"/>
+<!-- south -->
+<wire x1="56.134" y1="-5.9318" x2="-40.386" y2="-5.9318" width="0.2032" layer="20"/>
+<!-- west -->
+<wire x1="-56.134" y1="9.8612" x2="-56.134" y2="73.66" width="0.2032" layer="20"/>
+<!-- southwest -->
+<wire x1="-40.386" y1="-5.9318" x2="-56.134" y2="9.8612" width="0.2032" layer="20"/>
 <wire x1="33.21055625" y1="7.09435" x2="37.90355625" y2="7.09435" width="0.254" layer="20"/>
 <wire x1="33.21055625" y1="15.22235" x2="37.90355625" y2="15.22235" width="0.254" layer="20"/>
